Commit message: 修改URDF相关文件命名

File: src/zayv2_description/urdf/zayv2_description.urdf (robot description, URDF)
Before this commit: robot ZayV2-description, 7 links, 6 joints
Links:
- link base_link: geometry collision mesh filename=package://zayv2_description/meshes/base_link.stl; visual mesh filename=package://zayv2_description/meshes/base_link.stl
- link link1: geometry collision mesh filename=package://zayv2_description/meshes/link1.stl; visual mesh filename=package://zayv2_description/meshes/link1.stl
- link link2: geometry collision mesh filename=package://zayv2_description/meshes/link2.stl; visual mesh filename=package://zayv2_description/meshes/link2.stl
- link link3: geometry collision mesh filename=package://zayv2_description/meshes/link3.stl; visual mesh filename=package://zayv2_description/meshes/link3.stl
- link link4: geometry collision mesh filename=package://zayv2_description/meshes/link4.stl; visual mesh filename=package://zayv2_description/meshes/link4.stl
- link link5: geometry collision mesh filename=package://zayv2_description/meshes/link5.stl; visual mesh filename=package://zayv2_description/meshes/link5.stl
- link link6: geometry collision mesh filename=package://zayv2_description/meshes/link6.stl; visual mesh filename=package://zayv2_description/meshes/link6.stl

Commit message: feat(zayv2_description): 迁移到ROS 2并更新机器人描述包
- 将CMakeLists.txt从catkin迁移到ament_cmake，并添加正确的安装目标
- 创建详细的README.md文档，包含构建和启动说明
- 添加Python格式的launch文件，支持RViz2显示和Gazebo仿真
- 更新package.xml以支持ROS 2依赖关系和ament构建系统
- 移除ROS 1特有的配置文件和launch文件
- 更新URDF文件中的关节限制参数，提供实际的数值范围
- 添加RViz2配置文件用于机器人模型可视化
- 更新URDF注释信息，移除ROS 1特定的导出器信息

File: src/zayv2_description/urdf/zayv2_description.urdf (robot description, URDF)
Before this commit: robot zayv2_description, 7 links, 6 joints
Joints:
- joint joint1: limit lower=0 upper=0 effort=0 velocity=0 -> lower=-3.1415 upper=3.1415 effort=10.0 velocity=3.0
- joint joint2: limit lower=0 upper=0 effort=0 velocity=0 -> lower=-1.57075 upper=1.57075 effort=10.0 velocity=3.0
- joint joint3: limit lower=0 upper=0 effort=0 velocity=0 -> lower=-1.57075 upper=1.57075 effort=10.0 velocity=3.0
- joint joint4: limit lower=0 upper=0 effort=0 velocity=0 -> lower=-3.1415 upper=3.1415 effort=10.0 velocity=3.0
- joint joint5: limit lower=0 upper=0 effort=0 velocity=0 -> lower=-1.57075 upper=1.57075 effort=10.0 velocity=3.0; origin xyz=0 -0.029 0.11205 rpy=1.5708 -1.5708 0 -> xyz=0 -0.029 0.11205 rpy=-1.5708 -1.5708 0
- joint joint6: limit lower=0 upper=0 effort=0 velocity=0 -> lower=-3.1415 upper=3.1415 effort=10.0 velocity=3.0

Commit message: feat(arm_control): 更新关节5的初始位置和运动范围
- 将joint5的初始位置从1.47调整为1.5707（约π/2）
- 扩大link5关节的运动限制范围，下限从-1.57075调整为-1.88495，
上限从1.57075调整为1.88495，增加约±0.314弧度的运动范围

File: src/zayv2_description/urdf/zayv2_description.urdf (robot description, URDF)
Before this commit: robot zayv2_description, 7 links, 6 joints
Joints:
- joint joint5: limit lower=-1.57075 upper=1.57075 effort=10.0 velocity=3.0 -> lower=-1.88495 upper=1.88495 effort=10.0 velocity=3.0
